Commit message: Add Traj & Exec Generation support files

File: pc_support/urdf/pc_robot_wc1.xacro (robot description, xacro)
@@ -8,5 +8,5 @@
     <xacro:wc1 prefix=""/>
     <xacro:milling_tool prefix=""/>
-    <joint name="flange-mount_link" type="fixed">
+    <joint name="r3_flange-mount_link" type="fixed">
         <origin xyz="0 0 0" rpy="0 0 0"/>
         <parent link="r3_flange"/>
