Commit message: Update URDF

File: pc_support/urdf/milling_tool_macro.xacro (robot description, xacro)
@@ -5,7 +5,8 @@
     <link name="${prefix}mount_link">
         <visual>
-            <origin xyz="0 0 0" rpy="0 0 0" />
+            <origin xyz="0.0127 0 0" rpy="0 ${radians(90)} 0" />
             <geometry>
-                <mesh filename="package://pc_support/meshes/tool_visual.stl"/>
+                <cylinder radius="0.09525" length="0.0254"/>
+                <!-- <mesh filename="package://pc_support/meshes/tool_visual.stl"/> -->
             </geometry>
             <material name="tool">
@@ -14,13 +15,37 @@
         </visual>
         <collision>
-            <origin xyz="0 0 0" rpy="0 0 0" />
+            <origin xyz="0.0127 0 0" rpy="0 ${radians(90)} 0" />
             <geometry>
-                <mesh filename="package://pc_support/meshes/tool_collision.stl"/>
+                <cylinder radius="0.09525" length="0.0254"/>
+                <!-- <mesh filename="package://pc_support/meshes/tool_collision.stl"/> -->
             </geometry>
         </collision>
     </link>
+    <link name="${prefix}body">
+        <visual>
+            <origin xyz="0.0854 -0.03 0" rpy="${radians(90)} 0 0" />
+            <geometry>
+                <cylinder radius="0.06" length="0.2"/>
+            </geometry>
+            <material name="tool">
+                <color rgba="0.65 0.6 0.20 1"/>
+            </material>
+        </visual>
+        <collision>
+            <origin xyz="0.0854 -0.03 0" rpy="${radians(90)} 0 0" />
+            <geometry>
+                <cylinder radius="0.06" length="0.2"/>
+            </geometry>
+        </collision>
+    </link>
+    <!-- Visual Body Joints -->
+    <joint name="${prefix}mount_link-body" type="fixed">
+        <origin xyz="0 0 0" rpy="0 0 0"/>
+        <parent link="${prefix}mount_link"/>
+        <child link="${prefix}body"/>
+    </joint>
     <!-- TCP defined as the physical center-tip of the spray gun -->
     <joint name="${prefix}mount_link-mill_tcp" type="fixed">
-        <origin xyz="0.0889 0.1016 0" rpy="${radians(90)} 0 0"/>
+        <origin xyz="0.0889 0.1016 0" rpy="-${radians(90)} 0 0"/>
         <parent link="${prefix}mount_link"/>
         <child link="${prefix}mill_tcp"/>

File: pc_support/urdf/pc_robot_wc1.xacro (robot description, xacro)
@@ -2,9 +2,9 @@
 <robot name="pc_robot" xmlns:xacro="http://ros.org/wiki/xacro">
     <!-- Robot -->
-    <xacro:include filename="$(find motoman_mh50_support)/urdf/mh50_macro.xacro" />
+    <xacro:include filename="$(find aims_wc1_support)/urdf/wc1_macro.xacro" />
     <!-- End Effector -->
     <xacro:include filename="$(find pc_support)/urdf/milling_tool_macro.xacro" />
     <!-- Build Kinematic Chain using imported components -->
-    <xacro:motoman_mh50 prefix="r3_"/>
+    <xacro:wc1 prefix=""/>
     <xacro:milling_tool prefix=""/>
     <joint name="flange-mount_link" type="fixed">

Commit message: Fix URDF orientation

File: pc_support/urdf/milling_tool_macro.xacro (robot description, xacro)
@@ -47,5 +47,5 @@
     <!-- TCP defined as the physical center-tip of the spray gun -->
     <joint name="${prefix}mount_link-mill_tcp" type="fixed">
-        <origin xyz="0.0889 0.1016 0" rpy="-${radians(90)} 0 0"/>
+        <origin xyz="0.0889 0.1016 0" rpy="-${radians(90)} ${radians(180)} 0"/>
         <parent link="${prefix}mount_link"/>
         <child link="${prefix}mill_tcp"/>
